Commit message: Updating text, including example

File: description/urdf/1.urdf (robot description, URDF)
Before this commit: robot mybot, 1 links, 0 joints
Links:
- added link wheel; visual cylinder length=0.05 radius=0.1
- link base_link: geometry visual box size=0.5 0.5 0.5
Joints:
- added joint wheel_joint: type continuous, parent base_link, child wheel, origin xyz=0 -0.29 -0.3 rpy=1.5708 0 0, axis 0 1 0

Commit message: snapshot

File: description/urdf/1.urdf (robot description, URDF)
Before this commit: robot simple_robot, 2 links, 1 joints
Links:
- removed link wheel
- added link left_wheel; visual cylinder length=0.05 radius=0.1
- added link right_wheel; visual cylinder length=0.05 radius=0.1
- link base_link: geometry visual box size=0.5 0.5 0.25
Joints:
- added joint right_wheel_joint: type continuous, parent base_link, child right_wheel, origin xyz=0 0.29 -0.13 rpy=1.5708 0 0, axis 0 1 0
- joint wheel_joint: child wheel -> left_wheel; origin xyz=0 -0.29 -0.3 rpy=1.5708 0 0 -> xyz=0 -0.29 -0.13 rpy=1.5708 0 0
