Commit message: Renaming things, adding map layer content

File: description_2/urdf/3.urdf (robot description, URDF)
Before this commit: robot simple_robot, 3 links, 2 joints
Links:
- added link base_footprint; visual box size=1 1 0.001
- added link map; visual mesh filename=package://description_2/meshes/map1.dae
Joints:
- removed joint wheel_joint
- added joint base_footprint_joint: type fixed, parent base_link, child base_footprint, origin xyz=0 0 -0.23 rpy=0 0 0
- added joint left_wheel_joint: type continuous, parent base_link, child left_wheel, origin xyz=0 -0.29 -0.13 rpy=1.5708 0 0, axis 0 1 0
- added joint map_joint: type fixed, parent base_footprint, child map, origin xyz=0 0 0 rpy=0 0 0
