Commit message: Snapshot

File: description_2/urdf/2.urdf (robot description, URDF)
Before this commit: robot simple_robot, 5 links, 4 joints
Links:
- link base_footprint: geometry visual box size=0.5 0.5 0.001

File: description_2/urdf/3.urdf (robot description, URDF)
Before this commit: robot simple_robot, 5 links, 4 joints
Links:
- link base_footprint: geometry visual box size=0.5 0.5 0.001
